File: earring.kicad_sch (KiCad schematic)
At the start: 106 parts, among them J2 USB_C_Receptacle_USB2.0, Q1 NMOS 20V 0.75A 500mΩ@4.5V, Q2 NMOS 20V 0.75A 500mΩ@4.5V, Q3 NMOS 20V 0.75A 500mΩ@4.5V, Q4 NMOS 20V 0.75A 500mΩ@4.5V, Q5 light_sensor, U1 Magnetic Switch, U10 USBLC6-2P6, U20 LGS4056H, U24 SK9822-EC20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

Commit message: update stiffener layer
Other:
- note added: "Make sure C10 is close to pin 45 of RP2040"
- note added: "Make sure C12 is close to pin 44 of RP2040"
- note added: "R10 sets charging current 20k = 50 ma"
- note added: "TODO: TALK TO OPAL ABOUT CHARGE CURRENTS HERE"
- note added: "VBATT THROUGH RESISTOR TO CPU OKAY WHEN CPU IS UNPOWERED?"
- note removed: "MEASURE BATT VOLTAGE"
- note removed: "Make sure C10 is close to pin 44 of RP2040"
- note removed: "Make sure C8 is close to pin 45 of RP2040"
- note removed: "R8 sets charging current 10k = 100 ma"
- company: Twisted Fields LLC -> Sequoia Hope Alexander
- title: RP2040 Motor Controller -> RP2040 Earring
- moved on the sheet: C23, C25, C26, C29, C30, C33, Q5, R10, R8, U7
